Commit message: 修改了moveit_config,成功添加arm_hand并完成规划

File: arm5dof_description/urdf/arm5dof.urdf.xacro (robot description, xacro)
@@ -1,461 +1,250 @@
 <?xml version="1.0" encoding="utf-8"?>
 <!-- 五自由度机械臂 URDF模型  ROS版-->
-<robot
-  name="arm5dof">
-  <link
-    name="base_link">
-    <inertial>
-      <origin
-        xyz="-0.05549 -1.2443E-05 0.014047"
-        rpy="0 0 0" />
-      <mass
-        value="0.34831" />
-      <inertia
-        ixx="0.00037734"
-        ixy="-1.9667E-07"
-        ixz="-5.7059E-07"
-        iyy="0.0011827"
-        iyz="9.3336E-14"
-        izz="0.0015361" />
-    </inertial>
-    <visual>
-      <origin
-        xyz="0 0 0"
-        rpy="0 0 0" />
-      <geometry>
-        <mesh
-          filename="package://arm5dof_description/meshes/base_link.STL" />
-      </geometry>
-      <material
-        name="black">
-        <color
-          rgba="0.3 0.3 0.3 1" />
-      </material>
-    </visual>
-    <collision>
-      <origin
-        xyz="0 0 0"
-        rpy="0 0 0" />
-      <geometry>
-        <mesh
-          filename="package://arm5dof_description/meshes/base_link.STL" />
-      </geometry>
-    </collision>
-  </link>
-  <link
-    name="link1">
-    <inertial>
-      <origin
-        xyz="-0.0098047 1.4097E-06 0.014583"
-        rpy="0 0 0" />
-      <mass
-        value="0.047857" />
-      <inertia
-        ixx="9.9743E-06"
-        ixy="1.2606E-09"
-        ixz="5.9862E-07"
-        iyy="8.9062E-06"
-        iyz="2.193E-09"
-        izz="1.4861E-05" />
-    </inertial>
-    <visual>
-      <origin
-        xyz="0 0 0"
-        rpy="0 0 0" />
-      <geometry>
-        <mesh
-          filename="package://arm5dof_description/meshes/link1.STL" />
-      </geometry>
-      <material
-        name="green">
-        <color
-          rgba="0.6 0.6 0.6 1" />
-      </material>
-    </visual>
-    <collision>
-      <origin
-        xyz="0 0 0"
-        rpy="0 0 0" />
-      <geometry>
-        <mesh
-          filename="package://arm5dof_description/meshes/link1.STL" />
-      </geometry>
-    </collision>
-  </link>
-  <joint
-    name="joint1"
-    type="revolute">
-    <origin
-      xyz="0 0 0.052"
-      rpy="0 0 0" />
-    <parent
-      link="base_link" />
-    <child
-      link="link1" />
-    <axis
-      xyz="0 0 1" />
-    <limit
-      lower="-1.5708"
-      upper="1.5708"
-      effort="20"
-      velocity="3.5" />
-    <ros2_control>
-      <hardware_interface>
-        position_controllers/JointPositionController
-      </hardware_interface>
-    </ros2_control>
-  </joint>
-  <link
-    name="link2">
-    <inertial>
-      <origin
-        xyz="0.04 -5.5511E-17 6.7485E-17"
-        rpy="0 0 0" />
-      <mass
-        value="0.020202" />
-      <inertia
-        ixx="9.9386E-06"
-        ixy="1.7219E-08"
-        ixz="-5.3147E-21"
-        iyy="1.3724E-05"
-        iyz="-1.594E-21"
-        izz="5.1826E-06" />
-    </inertial>
-    <visual>
-      <origin
-        xyz="0 0 0"
-        rpy="0 0 0" />
-      <geometry>
-        <mesh
-          filename="package://arm5dof_description/meshes/link2.STL" />
-      </geometry>
-      <material
-        name="green">
-        <color
-          rgba="0 0.6 0 1" />
-      </material>
-    </visual>
-    <collision>
-      <origin
-        xyz="0 0 0"
-        rpy="0 0 0" />
-      <geometry>
-        <mesh
-          filename="package://arm5dof_description/meshes/link2.STL" />
-      </geometry>
-    </collision>
-  </link>
-  <joint
-    name="joint2"
-    type="revolute">
-    <origin
-      xyz="0 0 0.018"
-      rpy="-1.5708 0 0" />
-    <parent
-      link="link1" />
-    <child
-      link="link2" />
-    <axis
-      xyz="0 0 1" />
-    <limit
-      lower="-2.650"
-      upper="-0.2269"
-      effort="20"
-      velocity="3.5" />
-    <ros2_control>
-      <hardware_interface>
-        position_controllers/JointPositionController
-      </hardware_interface>
-    </ros2_control>
-  </joint>
-  <link
-    name="link3">
-    <inertial>
-      <origin
-        xyz="0.019908 0 -6.1294E-06"
-        rpy="0 0 0" />
-      <mass
-        value="0.050927" />
-      <inertia
-        ixx="1.2573E-05"
-        ixy="8.6095E-09"
-        ixz="-1.9789E-09"
-        iyy="1.7838E-05"
-        iyz="3.1614E-20"
-        izz="8.6328E-06" />
-    </inertial>
-    <visual>
-      <origin
-        xyz="0 0 0"
-        rpy="0 0 0" />
-      <geometry>
-        <mesh
-          filename="package://arm5dof_description/meshes/link3.STL" />
-      </geometry>
-      <material
-        name="gray">
-        <color
-          rgba="0.6 0.6 0.6 1" />
-      </material>
-    </visual>
-    <collision>
-      <origin
-        xyz="0 0 0"
-        rpy="0 0 0" />
-      <geometry>
-        <mesh
-          filename="package://arm5dof_description/meshes/link3.STL" />
-      </geometry>
-    </collision>
-  </link>
-  <joint
-    name="joint3"
-    type="revolute">
-    <origin
-      xyz="0.08 0 0"
-      rpy="0 0 0" />
-    <parent
-      link="link2" />
-    <child
-      link="link3" />
-    <axis
-      xyz="0 0 1" />
-    <limit
-      lower="-0.7854"
-      upper="1.5708"
-      effort="20"
-      velocity="3.5" />
-    <ros2_control>
-      <hardware_interface>
-        position_controllers/JointPositionController
-      </hardware_interface>
-    </ros2_control>
-  </joint>
-  <link
-    name="link4">
-    <inertial>
-      <origin
-        xyz="0.042216 0.0041806 -3.2915E-06"
-        rpy="0 0 0" />
-      <mass
-        value="0.094835" />
-      <inertia
-        ixx="2.4341E-05"
-        ixy="-2.5244E-06"
-        ixz="-1.9789E-09"
-        iyy="3.3312E-05"
-        iyz="1.4436E-20"
-        izz="3.0737E-05" />
-    </inertial>
-    <visual>
-      <origin
-        xyz="0 0 0"
-        rpy="0 0 0" />
-      <geometry>
-        <mesh
-          filename="package://arm5dof_description/meshes/link4.STL" />
-      </geometry>
-      <material
-        name="green">
-        <color
-          rgba="0 0.6 0 1" />
-      </material>
-    </visual>
-    <collision>
-      <origin
-        xyz="0 0 0"
-        rpy="0 0 0" />
-      <geometry>
-        <mesh
-          filename="package://arm5dof_description/meshes/link4.STL" />
-      </geometry>
-    </collision>
-  </link>
-  <joint
-    name="joint4"
-    type="revolute">
-    <origin
-      xyz="0.07615 0 0"
-      rpy="0 0 0" />
-    <parent
-      link="link3" />
-    <child
-      link="link4" />
-    <axis
-      xyz="0 0 1" />
-    <limit
-      lower="-1.5708"
-      upper="1.5708"
-      effort="20"
-      velocity="3.5" />
-    <ros2_control>
-      <hardware_interface>
-        position_controllers/JointPositionController
-      </hardware_interface>
-    </ros2_control>
-  </joint>
-  <link
-    name="link5">
-    <inertial>
-      <origin
-        xyz="-8.2184E-06 -0.0011968 0.01386"
-        rpy="0 0 0" />
-      <mass
-        value="0.049124" />
-      <inertia
-        ixx="8.2684E-06"
-        ixy="2.2759E-09"
-        ixz="5.1987E-11"
-        iyy="1.1645E-05"
-        iyz="5.9116E-07"
-        izz="1.5458E-05" />
-    </inertial>
-    <visual>
-      <origin
-        xyz="0 0 0"
-        rpy="0 0 0" />
-      <geometry>
-        <mesh
-          filename="package://arm5dof_description/meshes/link5.STL" />
-      </geometry>
-      <material
-        name="gray">
-        <color
-          rgba="0.6 0.6 0.6 1" />
-      </material>
-    </visual>
-    <collision>
-      <origin
-        xyz="0 0 0"
-        rpy="0 0 0" />
-      <geometry>
-        <mesh
-          filename="package://arm5dof_description/meshes/link5.STL" />
-      </geometry>
-    </collision>
-  </link>
-  <joint
-    name="joint5"
-    type="revolute">
-    <origin
-      xyz="0.0854 0 0"
-      rpy="-1.57079632679489 8.79419361882729E-05 -1.5707963267949" />
-    <parent
-      link="link4" />
-    <child
-      link="link5" />
-    <axis
-      xyz="0 0 1" />
-    <limit
-      lower="-1.5708"
-      upper="1.5708"
-      effort="20"
-      velocity="3.5" />
-    <ros2_control>
-      <hardware_interface>
-        position_controllers/JointPositionController
-      </hardware_interface>
-    </ros2_control>
-  </joint>
-  <link
-    name="left_gripper_link">
-    <inertial>
-      <origin
-        xyz="0.035118 0.00016366 5.5511E-17"
-        rpy="0 0 0" />
-      <mass
-        value="0.024589" />
-      <inertia
-        ixx="1.611E-06"
-        ixy="2.5381E-07"
-        ixz="1.1103E-20"
-        iyy="1.2951E-05"
-        iyz="-2.2806E-22"
-        izz="1.2364E-05" />
-    </inertial>
-    <visual>
-      <origin
-        xyz="0 0 0"
-        rpy="0 0 0" />
-      <geometry>
-        <mesh
-          filename="package://arm5dof_description/meshes/left_gripper_link.STL" />
-      </geometry>
-      <material
-        name="green">
-        <color
-          rgba="0 0.6 0 1" />
-      </material>
-    </visual>
-    <collision>
-      <origin
-        xyz="0 0 0"
-        rpy="0 0 0" />
-      <geometry>
-        <mesh
-          filename="package://arm5dof_description/meshes/left_gripper_link.STL" />
-      </geometry>
-    </collision>
-  </link>
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
Commit message: 调urdf零点,节点启动顺序

File: arm5dof_description/urdf/arm5dof.urdf.xacro (robot description, xacro)
@@ -81,9 +81,9 @@
   </link>
   <joint name="joint2" type="revolute">
-    <origin xyz="0 0 0.018" rpy="-1.5708 0 0" />
+    <origin xyz="0 0 0.018" rpy="-1.5708 -1.57 0" />
     <parent link="link1" />
     <child link="link2" />
     <axis xyz="0 0 1" />
-    <limit lower="-2.650" upper="-0.2269" effort="20" velocity="3.5" />
+    <limit lower="-1.57" upper="1.57" effort="20" velocity="3.5" />
     <ros2_control>
       <hardware_interface>

File: arm5dof_moveit_config/config/arm5dof.ros2_control.xacro (robot description, xacro)
@@ -1,54 +1,54 @@
 <?xml version="1.0"?>
 <robot xmlns:xacro="http://www.ros.org/wiki/xacro">
-    <xacro:macro name="arm5dof_ros2_control" params="name initial_positions_file">
-        <xacro:property name="initial_positions" value="${xacro.load_yaml(initial_positions_file)['initial_positions']}"/>
-        <ros2_control name="${name}" type="system">
-            <hardware>
-                <!-- By default, set up controllers for simulation. This won't work on real hardware -->
-                <plugin>mock_components/GenericSystem</plugin>
-            </hardware>
-            <joint name="joint1">
-                <command_interface name="position"/>
-                <state_interface name="position">
-                  <param name="initial_value">${initial_positions['joint1']}</param>
-                </state_interface>
-                <state_interface name="velocity"/>
-            </joint>
-            <joint name="joint2">
-                <command_interface name="position"/>
-                <state_interface name="position">
-                  <param name="initial_value">${initial_positions['joint2']}</param>
-                </state_interface>
-                <state_interface name="velocity"/>
-            </joint>
-            <joint name="joint3">
-                <command_interface name="position"/>
-                <state_interface name="position">
-                  <param name="initial_value">${initial_positions['joint3']}</param>
-                </state_interface>
-                <state_interface name="velocity"/>
-            </joint>
-            <joint name="joint4">
-                <command_interface name="position"/>
-                <state_interface name="position">
-                  <param name="initial_value">${initial_positions['joint4']}</param>
-                </state_interface>
-                <state_interface name="velocity"/>
-            </joint>
-            <joint name="joint5">
-                <command_interface name="position"/>
-                <state_interface name="position">
-                  <param name="initial_value">${initial_positions['joint5']}</param>
-                </state_interface>
-                <state_interface name="velocity"/>
-            </joint>
-            <joint name="left_gripper_joint">
-                <command_interface name="position"/>
-                <state_interface name="position">
-                  <param name="initial_value">${initial_positions['left_gripper_joint']}</param>
-                </state_interface>
-                <state_interface name="velocity"/>
-            </joint>
-        </ros2_control>
-    </xacro:macro>
+  <xacro:macro name="arm5dof_ros2_control" params="name initial_positions_file">
+    <xacro:property name="initial_positions" value="${xacro.load_yaml(initial_positions_file)['initial_positions']}"/>
+    <ros2_control name="${name}" type="system">
+      <hardware>
+        <!-- By default, set up controllers for simulation. This won't work on real hardware -->
+        <plugin>mock_components/GenericSystem</plugin>
+      </hardware>
+      <joint name="joint1">
+        <command_interface name="position"/>
+        <state_interface name="position">
+          <param name="initial_value">${initial_positions['joint1']}</param>
+        </state_interface>
+        <state_interface name="velocity"/>
+      </joint>
+      <joint name="joint2">
+        <command_interface name="position"/>
+        <state_interface name="position">
+          <param name="initial_value">${initial_positions['joint2']}</param>
+        </state_interface>
+        <state_interface name="velocity"/>
+      </joint>
+      <joint name="joint3">
+        <command_interface name="position"/>
+        <state_interface name="position">
+          <param name="initial_value">${initial_positions['joint3']}</param>
+        </state_interface>
+        <state_interface name="velocity"/>
+      </joint>
+      <joint name="joint4">
+        <command_interface name="position"/>
+        <state_interface name="position">
+          <param name="initial_value">${initial_positions['joint4']}</param>
+        </state_interface>
+        <state_interface name="velocity"/>
+      </joint>
+      <joint name="joint5">
+        <command_interface name="position"/>
+        <state_interface name="position">
+          <param name="initial_value">${initial_positions['joint5']}</param>
+        </state_interface>
+        <state_interface name="velocity"/>
+      </joint>
+      <joint name="left_gripper_joint">
+        <command_interface name="position"/>
+        <state_interface name="position">
+          <param name="initial_value">${initial_positions['left_gripper_joint']}</param>
+        </state_interface>
+        <state_interface name="velocity"/>
+      </joint>
+    </ros2_control>
+  </xacro:macro>
 </robot>

Commit message: 调整mtc任务阶段的逻辑、

File: arm5dof_description/urdf/arm5dof.urdf.xacro (robot description, xacro)
@@ -115,9 +115,9 @@
   </link>
   <joint name="joint3" type="revolute">
-    <origin xyz="0.08 0 0" rpy="0 0 0" />
+    <origin xyz="0 0 0" rpy="0 0 0" />
     <parent link="link2" />
     <child link="link3" />
     <axis xyz="0 0 1" />
-    <limit lower="-0.7854" upper="1.5708" effort="20" velocity="3.5" />
+    <limit lower="-1.5708" upper="1.5708" effort="20" velocity="3.5" />
     <ros2_control>
       <hardware_interface>

Commit message: 在什么空间规划?

File: arm5dof_description/urdf/arm5dof.urdf.xacro (robot description, xacro)
@@ -115,5 +115,5 @@
   </link>
   <joint name="joint3" type="revolute">
-    <origin xyz="0 0 0" rpy="0 0 0" />
+    <origin xyz="0.08 0 0" rpy="0 0 0" />
     <parent link="link2" />
     <child link="link3" />

Commit message: 设置目标点

File: arm5dof_description/urdf/arm5dof.urdf.xacro (robot description, xacro)
@@ -51,5 +51,5 @@
     <child link="link1" />
     <axis xyz="0 0 1" />
-    <limit lower="-1.5708" upper="1.5708" effort="20" velocity="3.5" />
+    <limit lower="-2.23" upper="2.23" effort="20" velocity="3.5" />
     <ros2_control>
       <hardware_interface>
@@ -119,5 +119,5 @@
     <child link="link3" />
     <axis xyz="0 0 1" />
-    <limit lower="-1.5708" upper="1.5708" effort="20" velocity="3.5" />
+    <limit lower="-2.55" upper="2.55" effort="20" velocity="3.5" />
     <ros2_control>
       <hardware_interface>
@@ -153,5 +153,5 @@
     <child link="link4" />
     <axis xyz="0 0 1" />
-    <limit lower="-1.5708" upper="1.5708" effort="20" velocity="3.5" />
+    <limit lower="-1.92" upper="2.55" effort="20" velocity="3.5" />
     <ros2_control>
       <hardware_interface>
@@ -187,5 +187,5 @@
     <child link="link5" />
     <axis xyz="0 0 1" />
-    <limit lower="-1.5708" upper="1.5708" effort="20" velocity="3.5" />
+    <limit lower="-3.14" upper="3.14" effort="20" velocity="3.5" />
     <ros2_control>
       <hardware_interface>
@@ -221,5 +221,5 @@
     <child link="left_gripper_link" />
     <axis xyz="0 0 1" />
-    <limit lower="0" upper="1.5708" effort="20" velocity="3.5" />
+    <limit lower="0" upper="2.0" effort="20" velocity="3.5" />
     <ros2_control>
       <hardware_interface>
@@ -291,6 +291,10 @@
     <child link="right_gripper_link" />
     <axis xyz="0 0 1" />
-    <limit lower="-1.5708" upper="0" effort="20" velocity="3.5" />
-    <mimic joint="left_gripper_joint" multiplier="-1" offset="0" />
+    <limit lower="-2.0" upper="0" effort="20" velocity="3.5" />
+    <ros2_control>
+      <hardware_interface>
+        position_controllers/JointPositionController
+      </hardware_interface>
+    </ros2_control>
   </joint>
   <link name="right_rubber_pad_link">
@@ -384,9 +388,55 @@
     <origin rpy="0.0 0.0 0.0" xyz="0.0 0.0 0.1" />
   </joint>
-  <!--添加世界坐标系到机械臂基坐标系的空间变换-->
+  <link name="body">
+    <inertial>
+      <origin xyz="0 0 0" rpy="0 0 0" />
+      <mass value="0.023734" />
+    </inertial>
+    <visual>
+      <origin xyz="-0.07 0 0.025" rpy="0 0 0" />
+      <geometry>
+        <box size="0.27 0.12 0.05"/>
+      </geometry>
+      <material name="black">
+        <color rgba="0.2 0.2 0.2 1"/>
+      </material>
+    </visual>
+    <collision>
+      <origin xyz="-0.1 0 0.025" rpy="0 0 0" />
+      <geometry>
+        <box size="0.3 0.2 0.05"/>
+      </geometry>
+    </collision>
+  </link>
+  <link name="body_left">
+    <inertial>
+      <origin xyz="0 0 0" rpy="0 0 0" />
+      <mass value="0.023734" />
+    </inertial>
+    <visual>
+      <origin xyz="-0.07 0 0.025" rpy="0 0 0" />
+      <geometry>
+        <box size="0.27 0.12 0.05"/>
+      </geometry>
+      <material name="black">
+        <color rgba="0.2 0.2 0.2 1"/>
+      </material>
+    </visual>
+    <collision>
+      <origin xyz="-0.1 0 0.025" rpy="0 0 0" />
+      <geometry>
+        <box size="0.3 0.2 0.05"/>
+      </geometry>
+    </collision>
+  </link>
+  <joint name="body_joint" type="fixed">
+    <parent link="body" />
+    <child link="base_link" />
+    <origin rpy="0.0 0.0 0.0" xyz="0.0 0.0 0.05" />
+  </joint>
   <link name="world" />
   <joint name="world_joint" type="fixed">
     <parent link="world" />
-    <child link="base_link" />
+    <child link="body" />
     <origin rpy="0.0 0.0 0.0" xyz="0.0 0.0 0.0" />
   </joint>

File: arm5dof_moveit_config/config/arm5dof.ros2_control.xacro (robot description, xacro)
@@ -50,4 +50,11 @@
         <state_interface name="velocity"/>
       </joint>
+      <joint name="right_gripper_joint">
+        <command_interface name="position"/>
+        <state_interface name="position">
+          <param name="initial_value">${initial_positions['right_gripper_joint']}</param>
+        </state_interface>
+        <state_interface name="velocity"/>
+      </joint>
     </ros2_control>
   </xacro:macro>

Commit message: 成功运行IKFast和mtc

File: arm5dof_description/urdf/arm5dof.urdf.xacro (robot description, xacro)
@@ -85,5 +85,5 @@
     <child link="link2" />
     <axis xyz="0 0 1" />
-    <limit lower="-1.57" upper="1.57" effort="20" velocity="3.5" />
+    <limit lower="-1.00" upper="1.36" effort="20" velocity="3.5" />
     <ros2_control>
       <hardware_interface>
@@ -373,13 +373,4 @@
       </material>
     </visual>
-    <collision>
-      <origin xyz="0 0 0" rpy="0 0 0" />
-      <geometry>
-        <sphere radius="0.005" />
-      </geometry>
-      <material name="plastic">
-        <color rgba="1.0 1.0 0.0 1" />
-      </material>
-    </collision>
   </link>
   <joint name="tool_center_joint" type="fixed">
@@ -388,55 +379,8 @@
     <origin rpy="0.0 0.0 0.0" xyz="0.0 0.0 0.1" />
   </joint>
-  <link name="body">
-    <inertial>
-      <origin xyz="0 0 0" rpy="0 0 0" />
-      <mass value="0.023734" />
-    </inertial>
-    <visual>
-      <origin xyz="-0.07 0 0.025" rpy="0 0 0" />
-      <geometry>
-        <box size="0.27 0.12 0.05"/>
-      </geometry>
-      <material name="black">
-        <color rgba="0.2 0.2 0.2 1"/>
-      </material>
-    </visual>
-    <collision>
-      <origin xyz="-0.1 0 0.025" rpy="0 0 0" />
-      <geometry>
-        <box size="0.3 0.2 0.05"/>
-      </geometry>
-    </collision>
-  </link>
-  <link name="body_left">
-    <inertial>
-      <origin xyz="0 0 0" rpy="0 0 0" />
-      <mass value="0.023734" />
-    </inertial>
-    <visual>
-      <origin xyz="-0.07 0 0.025" rpy="0 0 0" />
-      <geometry>
-        <box size="0.27 0.12 0.05"/>
-      </geometry>
-      <material name="black">
-        <color rgba="0.2 0.2 0.2 1"/>
-      </material>
-    </visual>
-    <collision>
-      <origin xyz="-0.1 0 0.025" rpy="0 0 0" />
-      <geometry>
-        <box size="0.3 0.2 0.05"/>
-      </geometry>
-    </collision>
-  </link>
-  <joint name="body_joint" type="fixed">
-    <parent link="body" />
-    <child link="base_link" />
-    <origin rpy="0.0 0.0 0.0" xyz="0.0 0.0 0.05" />
-  </joint>
   <link name="world" />
   <joint name="world_joint" type="fixed">
     <parent link="world" />
-    <child link="body" />
+    <child link="base_link" />
     <origin rpy="0.0 0.0 0.0" xyz="0.0 0.0 0.0" />
   </joint>
